File: DragonNTSC.kicad_sch (KiCad schematic)
At the start: 34 parts, among them IC1 74LS273N, IC2 MC6847, IC3 MC1372, IC4 NE555P, J2 Board Interconnect Male, J2 Video Output, Q161 2N4403, Q162 2N4401, Q3 2N3904

Commit message: move -5v
Connections:
- net -5V: now also J2.3 (Pin_3); no longer J2.2 (Pin_2)
Changed lines of the file:
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@@
   (no_connect (at 107.1372 58.7756))
   (no_connect (at 107.1372 48.6156))
-  (no_connect (at 255.0668 76.1492))
   (no_connect (at 145.288 47.3456))
   (no_connect (at 107.1372 61.3156))
@@
   (no_connect (at 107.1372 56.2356))
   (no_connect (at 107.1372 84.1756))
+  (no_connect (at 233.2228 35.0012))
   (no_connect (at 168.148 44.8056))
   (no_connect (at 107.1372 40.9956))
@@
       (effects (font (size 1.27 1.27)) hide)
     )
-    (pin "2")
-    (pin "1")
+    (pin "1")
+    (pin "2")
     (instances
       (project "DragonNTSC"
@@
       (effects (font (size 1.27 1.27)) hide)
     )
-    (pin "2")
-    (pin "1")
+    (pin "1")
+    (pin "2")
     (instances
       (project "DragonNTSC"
@@
       (effects (font (size 1.27 1.27)) hide)
     )
+    (pin "1")
+    (pin "8")
+    (pin "2")
     (pin "3")
     (pin "4")
-    (pin "1")
-    (pin "2")
-    (pin "8")
+    (pin "5")
     (pin "6")
-    (pin "5")
     (pin "7")
     (instances
@@
       (effects (font (size 1.27 1.27)) hide)
     )
-    (pin "2")
-    (pin "1")
+    (pin "1")
+    (pin "2")
     (instances
       (project "DragonNTSC"
@@
     )
   )
+  (symbol (lib_id "power:-5V") (at 255.0668 76.1492 270) (unit 1)
+    (in_bom yes) (on_board yes) (dnp no) (fields_autoplaced)
+    (property "Reference" "#PWR064" (at 257.6068 76.1492 0)
+      (effects (font (size 1.27 1.27)) hide)
+    )
+    (property "Value" "-5V" (at 258.8768 76.7842 90)
+      (effects (font (size 1.27 1.27)) (justify left))
+    )
+    (property "Footprint" "" (at 255.0668 76.1492 0)
+      (effects (font (size 1.27 1.27)) hide)
+    )
+    (property "Datasheet" "" (at 255.0668 76.1492 0)
+      (effects (font (size 1.27 1.27)) hide)
+    )
+    (pin "1")
+    (instances
+      (project "Dragon32"
+        (path "/0c3dceba-7c95-4b3d-b590-0eb581444beb"
+          (reference "#PWR064") (unit 1)
+        )
+      )
+      (project "DragonNTSC"
+        (path "/5c3ccdac-dbfc-47b7-be5c-593b42d2b61c"
+          (reference "#PWR04") (unit 1)
+        )
+      )
+    )
+  )
   (symbol (lib_id "power:GND") (at 83.0072 25.6286 270) (unit 1)
     (in_bom yes) (on_board yes) (dnp no)
@@
     )
   )
-  (symbol (lib_id "power:-5V") (at 233.2228 35.0012 270) (unit 1)
-    (in_bom yes) (on_board yes) (dnp no) (fields_autoplaced)
-    (property "Reference" "#PWR064" (at 235.7628 35.0012 0)
-      (effects (font (size 1.27 1.27)) hide)
-    )
-    (property "Value" "-5V" (at 237.0328 35.6362 90)
-      (effects (font (size 1.27 1.27)) (justify left))
-    )
-    (property "Footprint" "" (at 233.2228 35.0012 0)
-      (effects (font (size 1.27 1.27)) hide)
-    )
-    (property "Datasheet" "" (at 233.2228 35.0012 0)
-      (effects (font (size 1.27 1.27)) hide)
-    )
-    (pin "1")
-    (instances
-      (project "Dragon32"
-        (path "/0c3dceba-7c95-4b3d-b590-0eb581444beb"
-          (reference "#PWR064") (unit 1)
-        )
-      )
-      (project "DragonNTSC"
-        (path "/5c3ccdac-dbfc-47b7-be5c-593b42d2b61c"
-          (reference "#PWR04") (unit 1)
-        )
-      )
-    )
-  )
   (symbol (lib_id "power:GND") (at 91.8972 96.8756 0) (unit 1)
     (in_bom yes) (on_board yes) (dnp no) (fields_autoplaced)
@@
       (effects (font (size 1.27 1.27)) hide)
     )
+    (pin "1")
     (pin "2")
     (pin "3")
-    (pin "1")
     (instances
       (project "DragonNTSC"
@@
       (effects (font (size 1.27 1.27)) hide)
     )
-    (pin "2")
-    (pin "1")
+    (pin "1")
+    (pin "2")
     (instances
       (project "DragonNTSC"
@@
       (effects (font (size 1.27 1.27)) hide)
     )
-    (pin "2")
-    (pin "1")
-    (instances
-      (project "DragonNTSC"
+    (pin "1")
+    (pin "2")
+    (instances
+      (project "DragonNTSC"
