File: DragonNTSC.kicad_pcb (KiCad board)
At the start: 2 copper layers, 120.2 x 35.7 mm, 19 parts, among them IC1 74LS273N, IC2 MC6847, IC3 MC1372, J1 Video Output, J2 Board interconnect, Q1 2N4403, Q2 2N4401

Commit message: add missing css and fs lines
Parts:
- J2: value Board interconnect -> Board Interconnect Male; footprint Connector_PinHeader_2.54mm:PinHeader_2x10_P2.54mm_Vertical -> Connector_PinHeader_2.54mm:PinHeader_2x11_P2.54mm_Vertical
Connections:
- J2 pad 19: unconnected-(J2-Pin_19-Pad19) -> CSS
Routing:
- net CSS: track 0.00 -> 76.9 mm, vias 0 -> 1
- net ~{FS}: track 35.1 -> 101.6 mm, vias 2 -> 4
- net ~{A}/G: track 69.1 -> 73.5 mm
- net Net-(IC1-Q0): track 65.6 -> 68.3 mm, vias 1 -> 3
- net GM2: track 53.9 -> 51.7 mm
- net GND: track 255.5 -> 257.2 mm
- net DA0: track 51.0 -> 52.7 mm
- net GM1: track 56.5 -> 55.3 mm
- net Net-(IC1-Q7): track 78.0 -> 77.1 mm
- net Net-(IC1-Q5): track 43.2 -> 43.9 mm

Commit message: prototype experiment board
Parts:
- added C5: 0.1uF, Capacitor_SMD:C_0805_2012Metric, B.Cu at (95.9, 126.5)
- added C6: 0.1uF, Capacitor_SMD:C_0805_2012Metric, B.Cu at (132.8, 102.3)
- added C7: 0.1uF, Capacitor_SMD:C_0805_2012Metric, B.Cu at (161.5, 102.1)
- added IC4: 74LS273N, Package_DIP:DIP-20_W7.62mm, F.Cu at (110.0, 99.4)
- added IC5: 74LS273N, Package_DIP:DIP-20_W7.62mm, F.Cu at (138.7, 99.4)
- added J3: GPIO, Connector_PinHeader_2.54mm:PinHeader_2x20_P2.54mm_Vertical, F.Cu at (87.1, 86.4)
- added J4: Logic Analyser, Connector_PinHeader_2.54mm:PinHeader_2x16_P2.54mm_Vertical, F.Cu at (160.3, 86.2)
Connections:
- net Net-(IC1-Q0) renamed /D0
- net Net-(IC1-Q1) renamed /D1
- net Net-(IC1-Q2) renamed /D2
- net Net-(IC1-Q3) renamed /D3
- net Net-(IC1-Q4) renamed /D4
- net Net-(IC1-Q5) renamed /D5
- IC1 pad 11: ~{RAS0} -> RASEven
- IC1 pad 13: DO4 -> DP4
- IC1 pad 14: DO5 -> DP5
- IC1 pad 16: Net-(IC1-Q6) -> /D6
- IC1 pad 17: DO6 -> DP6
- IC1 pad 18: DO7 -> DP7
- IC1 pad 19: Net-(IC1-Q7) -> /D7
- IC1 pad 3: DO0 -> DP0
- IC1 pad 4: DO1 -> DP1
- IC1 pad 7: DO2 -> DP2
- IC1 pad 8: DO3 -> DP3
- IC2 pad 2: Net-(IC1-Q6) -> /D6
- IC2 pad 27: GM2 -> /GM2
- IC2 pad 29: GM1 -> /GM1
- IC2 pad 30: GM0 -> /GM0
- IC2 pad 31: GM0 -> /~{INT}/EXT
- IC2 pad 32: Net-(IC1-Q6) -> /INV
- IC2 pad 34: Net-(IC1-Q7) -> /~{A}/S
- IC2 pad 35: ~{A}/G -> /~{A}/G
- IC2 pad 39: CSS -> /CSS
- IC2 pad 40: Net-(IC1-Q7) -> /D7
- J2 pad 10: GM2 -> unconnected-(J2-Pin_10-Pad10)
- J2 pad 11: DO4 -> unconnected-(J2-Pin_11-Pad11)
- J2 pad 12: GM1 -> unconnected-(J2-Pin_12-Pad12)
- J2 pad 13: DO5 -> unconnected-(J2-Pin_13-Pad13)
- J2 pad 14: GM0 -> unconnected-(J2-Pin_14-Pad14)
- J2 pad 15: DO6 -> unconnected-(J2-Pin_15-Pad15)
- J2 pad 16: ~{RAS0} -> unconnected-(J2-Pin_16-Pad16)
- J2 pad 17: DO7 -> unconnected-(J2-Pin_17-Pad17)
- J2 pad 19: CSS -> unconnected-(J2-Pin_19-Pad19)
- J2 pad 20: ~{A}/G -> unconnected-(J2-Pin_20-Pad20)
- J2 pad 3: DO0 -> unconnected-(J2-Pin_3-Pad3)
- J2 pad 5: DO1 -> unconnected-(J2-Pin_5-Pad5)
- J2 pad 7: DO2 -> unconnected-(J2-Pin_7-Pad7)
- J2 pad 9: DO3 -> unconnected-(J2-Pin_9-Pad9)
Routing:
- net DP2: track 0.00 -> 144.9 mm, vias 0 -> 4
- net DP3: track 0.00 -> 143.7 mm, vias 0 -> 3
- net DA0: track 52.7 -> 172.8 mm, vias 1 -> 2
- net VCLK: track 115.7 -> 231.9 mm, vias 1 -> 2
- net DP1: track 0.00 -> 115.6 mm, vias 0 -> 4
- net DP4: track 0.00 -> 114.4 mm, vias 0 -> 1
- net DP0: track 0.00 -> 113.9 mm, vias 0 -> 6
- net RASEven: track 0.00 -> 113.1 mm, vias 0 -> 2
- net DP5: track 0.00 -> 101.3 mm, vias 0 -> 2
- net ~{FS}: track 101.6 -> 202.0 mm, vias 4 -> 7
- net ~{HS}: track 86.7 -> 181.2 mm, vias 1 -> 3
- net DP6: track 0.00 -> 92.5 mm, vias 0 -> 2
- net DP7: track 0.00 -> 85.9 mm, vias 0 -> 2
- net Net-(IC1-Q7): track 77.1 -> 0.00 mm, vias 2 -> 0
- net CSS: track 76.9 -> 0.00 mm, vias 1 -> 0
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Other:
- board size 120.2 x 35.7 mm -> 120.2 x 54.2 mm
- board text added: "-"
- board text added: "GND"
- board text added: "GPIO"
- board text added: "Logic Analyser"

Commit message: refine board
Parts:
- added JP1: Jumper_3_Open, Connector_PinHeader_2.54mm:PinHeader_1x03_P2.54mm_Vertical, F.Cu at (145.8, 81.9)
- added JP2: Jumper_3_Open, Connector_PinHeader_2.54mm:PinHeader_1x03_P2.54mm_Vertical, F.Cu at (145.8, 85.5)
Connections:
- IC5 pad 11: RASEven -> RAScontrol
- J3 pad 19: unconnected-(J3-Pin_19-Pad19) -> RASSpare
- J4 pad 19: unconnected-(J4-Pin_19-Pad19) -> RAScontrol
- J4 pad 21: unconnected-(J4-Pin_21-Pad21) -> RASEven
Routing:
- net RASSpare: track 0.00 -> 42.5 mm, vias 0 -> 2
- net RASEven: track 113.1 -> 155.5 mm, vias 2 -> 3
- net RAScontrol: track 0.00 -> 40.6 mm
- net RASOdd: track 27.5 -> 41.9 mm
- net ~{FS}: track 202.0 -> 192.0 mm, vias 7 -> 6
- net Net-(JP1-C): track 0.00 -> 4.68 mm
- net /D0: track 68.2 -> 67.5 mm, vias 3 -> 2
- net /D6: track 56.5 -> 57.2 mm
- net DP7: track 85.9 -> 86.5 mm
- net DP3: track 143.7 -> 143.2 mm
- net DP5: track 101.3 -> 100.8 mm
- net DP4: track 114.4 -> 113.9 mm
- net DP2: track 144.9 -> 144.4 mm
- net GND: vias 45 -> 44
Other:
- board text added: "+5V"
- board text added: "CHB"
- board text added: "CSS"
- board text added: "D0"
- board text added: "D1"
- board text added: "D2"
- board text added: "D3"
- board text added: "D4"
- board text added: "D5"
- board text added: "D6"
- board text added: "D7"
- board text added: "DA0"
- board text added: "GM0"
- board text added: "GM1"
- board text added: "GM2"
- board text added: "INV"
- board text added: "VCLK"
- board text added: "Y"
- board text added: "~{A}/G"
- board text added: "~{A}/S"
- board text added: "~{FS}"
- board text added: "~{HS}"
- board text added: "~{INT} /EXT"
- board text added: "~{MS}"
- board text added: "øA"
- board text added: "øB"

Commit message: add decoration
Parts:
- moved C1 0.27 mm to (120.6, 104.3)
Other:
- board text added: "BUFFER"
- board text added: "CONTROL"
- board text added: "DATA"
- board text added: "EVEN"
- board text added: "ODD"
- board text added: "SPARE"
